File: hardware/shield_v03/wat.kicad_pcb (KiCad board)
At the start: 2 copper layers, 36 parts, among them J1 GS2, J2 GS2, J3 GS2, J4 Conn_02x05_Odd_Even, P1 V_IN, P2 PINZA_1, P3 PINZA_2, P4 PINZA_3, P5 PINZA_4, P6 PINZA_5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

Commit message: desarrollo hardware
Parts:
- added C12: 100nF, Capacitors_SMD:C_1206_HandSoldering, F.Cu at (109.0, 89.0)
- added C13: 100nF, Capacitors_SMD:C_1206_HandSoldering, F.Cu at (77.8, 88.8)
- added R11: 4K7, Resistors_SMD:R_2512_HandSoldering, F.Cu at (114.0, 91.0)
- added R12: 4K7, Resistors_SMD:R_2512_HandSoldering, F.Cu at (98.8, 91.2)
- added R13: 4K7, Resistors_SMD:R_2512_HandSoldering, F.Cu at (83.0, 90.8)
- moved R1 126.4 mm to (153.2, 112.2)
- moved R2 125.8 mm to (153.0, 125.8)
- moved D1 108.4 mm to (142.6, 73.4)
- moved P1 108.4 mm to (142.6, 62.2)
- moved C1 108.2 mm to (145.5, 126.0)
- moved C5 106.8 mm to (135.8, 111.8), turned to 90 degrees
- moved C4 105.4 mm to (146.0, 85.0)
- moved U1 105.1 mm to (145.0, 112.0), turned to 90 degrees
- moved J1 69.1 mm to (108.2, 96.8)
- moved J3 68.7 mm to (77.2, 96.0)
- moved J2 68.6 mm to (93.0, 97.0)
- moved J4 57.7 mm to (76.5, 75.8)
- moved U2 56.0 mm to (89.2, 112.0)
- moved C10 45.3 mm to (93.5, 89.2), turned to 90 degrees
- moved R3 41.6 mm to (72.2, 138.5)
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Connections:
- C10 pad 1: /ss -> /esp_d1

Commit message: avance en pcb
Parts:
- moved W1 81.2 mm to (108.6, 101.3)
- moved P8 79.9 mm to (107.1, 79.1), turned to 180 degrees
- moved C7 63.2 mm to (105.2, 88.6), turned to 90 degrees
- moved R6 52.9 mm to (101.5, 96.8), turned to 90 degrees
- moved U1 31.0 mm to (114.0, 110.1)
- moved R1 28.7 mm to (124.7, 108.8)
- moved C4 28.5 mm to (120.1, 97.0), turned to 180 degrees
- moved R2 28.4 mm to (124.7, 123.6)
- moved C5 27.7 mm to (110.9, 124.0), turned to 270 degrees
- moved C1 27.6 mm to (118.0, 124.1)
- moved P1 26.5 mm to (122.3, 79.2), turned to 180 degrees
- moved D1 25.4 mm to (122.3, 88.5)
- moved J1 22.6 mm to (86.1, 101.5)
- moved R11 20.5 mm to (93.5, 91.6)
- moved C12 20.4 mm to (89.2, 93.9)
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Connections:
- C12 pad 1: /esp_d0 -> /esp_d2
- C13 pad 1: /esp_d2 -> /esp_d0
- J1 pad 2: /esp_d0 -> /esp_d2
- J3 pad 2: /esp_d2 -> /esp_d0
- J4 pad 10: GND -> /miso
- J4 pad 2: /mosi -> /esp_d2
- J4 pad 3: /esp_d0 -> /esp_d8
- J4 pad 4: /miso -> /esp_d1
- J4 pad 5: /esp_d1 -> /esp_d3
- J4 pad 6: /sck -> /esp_d0
- J4 pad 7: /esp_d2 -> GND
- J4 pad 8: /esp_d8 -> /mosi
- J4 pad 9: /esp_d3 -> /sck
- R11 pad 2: /esp_d0 -> /esp_d2
- R13 pad 2: /esp_d2 -> /esp_d0
Routing:
- net /v_referencia: track 0.00 -> 249.2 mm
- net VCC: track 0.00 -> 68.0 mm
- net /intensidad_6: track 0.00 -> 66.8 mm
- net /intensidad_5: track 0.00 -> 60.6 mm
- net /intensidad_7: track 0.00 -> 59.1 mm
- net /vcc_5v: track 0.00 -> 56.5 mm
- net /intensidad_4: track 0.00 -> 54.8 mm
- net /sck: track 0.00 -> 48.0 mm
- net /intensidad_3: track 0.00 -> 46.7 mm
- net /esp_d2: track 0.00 -> 42.0 mm
- net /intensidad_2: track 0.00 -> 41.1 mm
- net /intensidad_1: track 0.00 -> 38.2 mm
- net /esp_d1: track 0.00 -> 29.4 mm
- net /esp_d0: track 0.00 -> 29.4 mm
- net /mosi: track 0.00 -> 28.5 mm
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