File: hardware/shield_v03/wat.kicad_pcb (KiCad board)
At the start: 2 copper layers, 42 parts, among them J1 GS2, J2 GS2, J3 GS2, J4 Conn_02x05, J5 Conn_02x05, P1 V_IN, P2 PINZA_1, P3 PINZA_2, P4 PINZA_3, P5 PINZA_4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

Commit message: desarrollo hardware
Parts:
- removed C7: 100nF, Capacitors_SMD:C_1206_HandSoldering
- added R10: 10k, Resistors_SMD:R_1206_HandSoldering, F.Cu at (103.5, 88.5)
- J4, J5: value Conn_02x05 -> Conn_02x05_Odd_Even
- R1, R11, R12, R13, R2: footprint Resistors_SMD:R_2512_HandSoldering -> Resistors_SMD:R_1206_HandSoldering
- R6: value 10k -> 1k
- moved W1 10.2 mm to (125.8, 97.0)
- moved C13 4.08 mm to (73.2, 91.2)
- moved C10 4.06 mm to (82.8, 91.2)
- moved C12 4.04 mm to (92.2, 91.2)
- moved J1 3.55 mm to (88.4, 98.7)
- moved J2 3.55 mm to (84.5, 98.7)
- moved J3 3.55 mm to (80.7, 98.7)
- moved R12 2.45 mm to (86.2, 91.2)
- moved R2 2.43 mm to (124.0, 121.2)
- moved R1 2.38 mm to (124.0, 106.5)
- moved R13 2.35 mm to (76.8, 91.2)
- moved R11 2.30 mm to (95.8, 91.2)
- moved C1 1.35 mm to (117.8, 122.8)
- moved C5 1.27 mm to (110.6, 122.7)
- moved U1 0.87 mm to (116.8, 105.2)
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Connections:
- P8 pad 2: /intensidad_7 -> Net-(P8-Pad2)
- R6 pad 1: /intensidad_7 -> /voltage_1
- U2 pad 25: /intensidad_7 -> /voltage_1
Routing:
- net /v_referencia: track 0.00 -> 288.3 mm
- net VCC: track 0.00 -> 70.7 mm
- net /sck: track 0.00 -> 67.2 mm
- net /intensidad_6: track 0.00 -> 62.4 mm
- net /intensidad_5: track 0.00 -> 56.8 mm
- net /intensidad_4: track 0.00 -> 50.5 mm
- net /esp_d2: track 0.00 -> 47.4 mm
- net /voltage_1: track 0.00 -> 47.0 mm
- net /intensidad_3: track 0.00 -> 43.6 mm
- net /intensidad_1: track 0.00 -> 43.1 mm
- net /intensidad_2: track 0.00 -> 40.1 mm
- net /esp_d1: track 0.00 -> 28.6 mm
- net Net-(C1-Pad1): track 0.00 -> 27.5 mm
- net /mosi: track 0.00 -> 25.9 mm
- net /miso: track 0.00 -> 25.9 mm
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Other:
- board outline added: 67.2 x 86.2 mm

Commit message: primera version hardware esclavo
Parts:
- moved C13 2.35 mm to (73.2, 93.6)
- moved C12 2.35 mm to (92.2, 93.6)
- moved C10 2.29 mm to (82.8, 93.5)
- moved J1 2.29 mm to (88.4, 101.0)
- moved J2 2.29 mm to (84.5, 101.0)
- moved J3 2.29 mm to (80.7, 101.0)
- moved R11 2.29 mm to (95.8, 93.5)
- moved R12 2.29 mm to (86.2, 93.5)
- moved R13 2.29 mm to (76.8, 93.5)
- moved W1 1.94 mm to (124.0, 96.3)
Connections:
- C1 pad 1: Net-(C1-Pad1) -> /v_25
- R1 pad 2: Net-(C1-Pad1) -> /v_25
- R2 pad 1: Net-(C1-Pad1) -> /v_25
- U1 pad 3: Net-(C1-Pad1) -> /v_25
- U1 pad 5: (no net) -> /v_25
- U1 pad 6: (no net) -> Net-(U1-Pad6)
- U1 pad 7: (no net) -> Net-(U1-Pad6)
Routing:
- net GND: track 0.00 -> 264.4 mm, vias 0 -> 5
- net VCC: track 70.7 -> 123.7 mm, vias 0 -> 4
- net /vcc_5v: track 6.96 -> 51.2 mm
- net /v_25: track 0.00 -> 35.4 mm
- net Net-(C1-Pad1): track 27.5 -> 0.00 mm
- net /esp_d0: track 24.1 -> 49.2 mm, vias 0 -> 1
- net /mosi: track 25.9 -> 48.0 mm, vias 0 -> 1
- net /miso: track 25.9 -> 46.8 mm, vias 0 -> 1
- net /esp_d1: track 28.6 -> 48.9 mm, vias 0 -> 1
- net Net-(U1-Pad6): track 0.00 -> 7.61 mm
- net /esp_d2: track 47.4 -> 49.9 mm
- net /v_referencia: track 288.3 -> 286.6 mm
- net /ss: track 22.1 -> 20.4 mm
- net /sck: track 67.2 -> 67.5 mm, vias 0 -> 1

Commit message: primera version del esclavo terminada
Routing:
- net GND: track 264.4 -> 405.0 mm, vias 5 -> 17
- added copper zone on B.Cu, net GND
- added copper zone on F.Cu, net GND
Changed lines of the file:
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@@
-(kicad_pcb (version 4) (host pcbnew 4.0.7-e2-6376~61~ubuntu18.04.1)
+(kicad_pcb (version 4) (host pcbnew 4.0.2+dfsg1-stable)
   (general
     (links 91)
     (no_connects 0)
-    (area 60.674999 73.924999 128.075001 160.325001)
+    (area 19.384287 33.726 197.585001 208.313001)
     (thickness 1.6)
-    (drawings 50)
-    (tracks 347)
+    (drawings 51)
+    (tracks 405)
     (zones 0)
     (modules 42)
@@
   )
   (setup
-    (last_trace_width 0.25)
+    (last_trace_width 0.8)
     (user_trace_width 0.4)
     (user_trace_width 0.6)
@@
     )
   )
+  (gr_line (start 69.25 138.5) (end 122.5 138.5) (angle 90) (layer Dwgs.User) (width 0.2))
   (gr_line (start 197.485 122.174) (end 197.485 120.142) (angle 90) (layer Dwgs.User) (width 0.2))
   (gr_line (start 152.781 122.174) (end 197.485 122.174) (angle 90) (layer Dwgs.User) (width 0.2))
@@
     (arrow2b (pts (xy 35.306 160.274) (xy 34.719579 159.147496)))
   )
+  (segment (start 91.25 115.824) (end 91.25 115.75) (width 0.8) (layer B.Cu) (net 1))
+  (segment (start 93 114) (end 94 113) (width 0.8) (layer F.Cu) (net 1))
+  (via (at 93 114) (size 0.6) (drill 0.4) (layers F.Cu B.Cu) (net 1))
+  (segment (start 91.25 115.75) (end 93 114) (width 0.8) (layer B.Cu) (net 1))
+  (segment (start 103.5 115.824) (end 103.5 115.75) (width 0.8) (layer B.Cu) (net 1))
+  (segment (start 105.25 114) (end 106 113.25) (width 0.8) (layer F.Cu) (net 1))
+  (via (at 105.25 114) (size 0.6) (drill 0.4) (layers F.Cu B.Cu) (net 1))
+  (segment (start 103.5 115.75) (end 105.25 114) (width 0.8) (layer B.Cu) (net 1))
+  (segment (start 62.992 82.5) (end 78 82.5) (width 0.8) (layer B.Cu) (net 1))
+  (segment (start 78 82.5) (end 79.25 81.25) (width 0.8) (layer F.Cu) (net 1))
+  (via (at 78 82.5) (size 0.6) (drill 0.4) (layers F.Cu B.Cu) (net 1))
+  (segment (start 63.102 127.5) (end 63.102 130.148) (width 1.2) (layer B.Cu) (net 1))
+  (segment (start 63 130.25) (end 63 132.75) (width 1.2) (layer F.Cu) (net 1))
+  (via (at 63 130.25) (size 0.6) (drill 0.4) (layers F.Cu B.Cu) (net 1))
+  (segment (start 63.102 130.148) (end 63 130.25) (width 1.2) (layer B.Cu) (net 1))
+  (segment (start 117.25 133.75) (end 117.5 133.75) (width 1.2) (layer B.Cu) (net 1))
+  (segment (start 112 133.75) (end 117.25 133.75) (width 1.2) (layer B.Cu) (net 1))
+  (segment (start 119.75 136) (end 122.25 138.5) (width 1.2) (layer F.Cu) (net 1))
+  (via (at 119.75 136) (size 0.6) (drill 0.4) (layers F.Cu B.Cu) (net 1))
+  (segment (start 117.5 133.75) (end 119.75 136) (width 1.2) (layer B.Cu) (net 1))
+  (segment (start 112 133.75) (end 112 136) (width 1.2) (layer B.Cu) (net 1))
+  (segment (start 112 136) (end 112 138.5) (width 1.2) (layer F.Cu) (net 1))
+  (via (at 112 136) (size 0.6) (drill 0.4) (layers F.Cu B.Cu) (net 1))
+  (segment (start 101.5 133.75) (end 101.5 136) (width 1.2) (layer B.Cu) (net 1))
+  (segment (start 101.5 136) (end 101.5 138.5) (width 1.2) (layer F.Cu) (net 1))
+  (via (at 101.5 136) (size 0.6) (drill 0.4) (layers F.Cu B.Cu) (net 1))
+  (segment (start 90.75 133.75) (end 90.75 136) (width 1.2) (layer B.Cu) (net 1))
+  (segment (start 90.75 136) (end 90.75 138.5) (width 1.2) (layer F.Cu) (net 1))
+  (via (at 90.75 136) (size 0.6) (drill 0.4) (layers F.Cu B.Cu) (net 1))
+  (segment (start 80.5 133.75) (end 80.5 136) (width 1.2) (layer B.Cu) (net 1))
+  (segment (start 80.5 136) (end 80.5 138.5) (width 1.2) (layer F.Cu) (net 1))
+  (via (at 80.5 136) (size 0.6) (drill 0.4) (layers F.Cu B.Cu) (net 1))
+  (segment (start 72 133.75) (end 72 136) (width 1.2) (layer B.Cu) (net 1))
+  (segment (start 72 136) (end 72 138.5) (width 1.2) (layer F.Cu) (net 1))
+  (via (at 72 136) (size 0.6) (drill 0.4) (layers F.Cu B.Cu) (net 1))
+  (segment (start 63.102 113.648) (end 63.102 127.5) (width 1.2) (layer B.Cu) (net 1))
+  (segment (start 63.102 127.5) (end 63.102 127.852) (width 1.2) (layer B.Cu) (net 1))
+  (segment (start 108.75 133.75) (end 112 133.75) (width 1.2) (layer B.Cu) (net 1))
+  (segment (start 99.75 133.75) (end 101.5 133.75) (width 1.2) (layer B.Cu) (net 1))
+  (segment (start 101.5 133.75) (end 108.75 133.75) (width 1.2) (layer B.Cu) (net 1))
+  (segment (start 69 133.75) (end 72 133.75) (width 1.2) (layer B.Cu) (net 1))
+  (segment (start 72 133.75) (end 80.5 133.75) (width 1.2) (layer B.Cu) (net 1))
+  (segment (start 80.5 133.75) (end 90.75 133.75) (width 1.2) (layer B.Cu) (net 1))
+  (segment (start 90.75 133.75) (end 99.75 133.75) (width 1.2) (layer B.Cu) (net 1))
+  (segment (start 63.102 127.852) (end 69 133.75) (width 1.2) (layer B.Cu) (net 1))
+  (segment (start 69.25 89.281) (end 69.25 91.75) (width 0.6) (layer B.Cu) (net 1))
+  (segment (start 69.25 91.75) (end 69.25 93.75) (width 0.6) (layer F.Cu) (net 1))
+  (via (at 69.25 91.75) (size 0.6) (drill 0.4) (layers F.Cu B.Cu) (net 1))
+  (segment (start 66.75 89.281) (end 66.75 91.75) (width 0.6) (layer B.Cu) (net 1))
+  (segment (start 66.75 91.75) (end 66.75 93.75) (width 0.6) (layer F.Cu) (net 1))
+  (via (at 66.75 91.75) (size 0.6) (drill 0.4) (layers F.Cu B.Cu) (net 1))
   (segment (start 73.152 91.599) (end 73.152 90.297) (width 0.6) (layer F.Cu) (net 1))
   (via (at 72.136 89.281) (size 0.6) (drill 0.4) (layers F.Cu B.Cu) (net 1))
@@
   (segment (start 91.44 89.281) (end 82.042 89.281) (width 0.6) (layer B.Cu) (net 1))
   (segment (start 66.421 89.281) (end 62.992 92.71) (width 0.6) (layer B.Cu) (net 1))
-  (segment (start 72.136 89.281) (end 66.421 89.281) (width 0.6) (layer B.Cu) (net 1))
+  (segment (start 72.136 89.281) (end 69.25 89.281) (width 0.6) (layer B.Cu) (net 1))
+  (segment (start 69.25 89.281) (end 66.75 89.281) (width 0.6) (layer B.Cu) (net 1))
+  (segment (start 66.75 89.281) (end 67 89.281) (width 0.6) (layer B.Cu) (net 1))
+  (segment (start 67 89.281) (end 66.421 89.281) (width 0.6) (layer B.Cu) (net 1))
   (segment (start 82.042 89.281) (end 75.057 89.281) (width 0.6) (layer B.Cu) (net 1))
   (segment (start 75.057 89.281) (end 72.136 89.281) (width 0.6) (layer B.Cu) (net 1))
@@
   (segment (start 89.154 75.184) (end 118.237 75.184) (width 1.2) (layer B.Cu) (net 1))
   (segment (start 118.237 75.184) (end 122.301 79.248) (width 1.2) (layer B.Cu) (net 1))
-  (segment (start 101.346 115.824) (end 65.278 115.824) (width 1.2) (layer B.Cu) (net 1))
-  (segment (start 65.278 115.824) (end 62.992 113.538) (width 1.2) (layer B.Cu) (net 1))
+  (segment (start 101.346 115.824) (end 91.25 115.824) (width 1.2) (layer B.Cu) (net 1))
+  (segment (start 91.25 115.824) (end 65.278 115.824) (width 1.2) (layer B.Cu) (net 1))
+  (segment (start 65.278 115.824) (end 63.102 113.648) (width 1.2) (layer B.Cu) (net 1))
+  (segment (start 63.102 113.648) (end 62.992 113.538) (width 1.2) (layer B.Cu) (net 1))
   (segment (start 62.992 113.538) (end 62.992 92.71) (width 1.2) (layer B.Cu) (net 1))
   (segment (start 68.072 76.835) (end 68.072 77.724) (width 1.2) (layer B.Cu) (net 1))
-  (segment (start 62.992 92.71) (end 62.992 76.327) (width 1.2) (layer B.Cu) (net 1))
+  (segment (start 62.992 92.71) (end 62.992 82.5) (width 1.2) (layer B.Cu) (net 1))
+  (segment (start 62.992 82.5) (end 62.992 76.327) (width 1.2) (layer B.Cu) (net 1))
   (segment (start 62.992 76.327) (end 63.881 75.438) (width 1.2) (layer B.Cu) (net 1))
   (segment (start 63.881 75.438) (end 66.675 75.438) (width 1.2) (layer B.Cu) (net 1))
@@
   (via (at 118.618 111.633) (size 0.6) (drill 0.4) (layers F.Cu B.Cu) (net 1))
   (segment (start 118.618 111.633) (end 114.427 115.824) (width 1.2) (layer B.Cu) (net 1))
-  (segment (start 114.427 115.824) (end 102.87 115.824) (width 1.2) (layer B.Cu) (net 1))
+  (segment (start 114.427 115.824) (end 103.5 115.824) (width 1.2) (layer B.Cu) (net 1))
+  (segment (start 103.5 115.824) (end 102.87 115.824) (width 1.2) (layer B.Cu) (net 1))
   (segment (start 99.24 117.803) (end 99.24 121.12) (width 1.2) (layer B.Cu) (net 1))
   (segment (start 102.87 115.824) (end 101.346 115.824) (width 1.2) (layer B.Cu) (net 1))
@@
   (segment (start 116.84 98.044) (end 116.713 98.044) (width 0.6) (layer F.Cu) (net 42))
   (segment (start 117.385 98.589) (end 116.84 98.044) (width 0.6) (layer F.Cu) (net 42))
+  (zone (net 1) (net_name GND) (layer F.Cu) (hatch edge 0.508)
+    (connect_pads (clearance 0.508))
+    (min_thickness 0.254)
+    (fill yes (arc_segments 16) (thermal_gap 0.508) (thermal_bridge_width 0.508))
+    (polygon
+      (pts
+        (xy 128 160.25) (xy 60.75 160.25) (xy 60.75 74) (xy 128 74) (xy 128 160.25)
+      )
+    )
+  )
+  (zone (net 1) (net_name GND) (layer B.Cu) (hatch edge 0.508)
+    (connect_pads (clearance 0.508))
+    (min_thickness 0.254)
+    (fill yes (arc_segments 16) (thermal_gap 0.508) (thermal_bridge_width 0.508))
+    (polygon
+      (pts
+        (xy 128 160.25) (xy 60.75 160.25) (xy 60.75 74) (xy 128 74) (xy 128 160.25)
+      )
+    )
+  )
 )
