File: hardware/shield_v03/wat.sch (KiCad schematic (older format))
At the start: 36 parts, among them J1 GS2, J2 GS2, J3 GS2, J4 Conn_02x05_Odd_Even, P1 V_IN, P2 PINZA_1, P3 PINZA_2, P4 PINZA_3, P5 PINZA_4, P6 PINZA_5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

Commit message: sincronizacion varios registros
Parts:
- C1, C4, C5: footprint Capacitors_THT:CP_Radial_D5.0mm_P2.00mm -> Capacitors_SMD:C_2220_HandSoldering
- C10, C11, C2, C3, C6, C7, C8, C9: footprint Capacitors_THT:C_Disc_D5.0mm_W2.5mm_P5.00mm -> Capacitors_SMD:C_1206_HandSoldering
- D1: footprint Diodes_ThroughHole:Diode_DO-35_SOD27_Horizontal_RM10 -> Diodes_SMD:D_2114
- J4: footprint (none) -> Pin_Headers:Pin_Header_Straight_2x05_Pitch2.54mm
- P1, P2, P3, P4, P5, P6, P7, P8: footprint Connect:bornier2 -> Connectors_Terminal_Blocks:TerminalBlock_bornier-2_P5.08mm
- R1, R2: value R -> 4K7; footprint (none) -> Resistors_SMD:R_2512_HandSoldering
- R3, R4, R5, R6, R7, R8, R9: footprint Resistors_ThroughHole:Resistor_Horizontal_RM10mm -> libreria_huellas_proyecto:Resistor_Horizontal_RM10mm
- U1: footprint (none) -> Housings_SOIC:SO-8_5.3x6.2mm_Pitch1.27mm
- U2: footprint oscar_libreria_huellas:arduino_nano -> libreria_huellas_proyecto:arduino_nano
Changed lines of the file:
@@
 LIBS:contrib
 LIBS:valves
+LIBS:recom-rd
+LIBS:RO-1224S
+LIBS:mp-1584
+LIBS:nano
 LIBS:wat-cache
 EELAYER 25 0
@@
 F 0 "P2" H 1195 5775 50  0000 C CNN
 F 1 "PINZA_1" V 1295 5625 50  0000 C CNN
-F 2 "Connect:bornier2" H 1195 5625 50  0001 C CNN
+F 2 "Connectors_Terminal_Blocks:TerminalBlock_bornier-2_P5.08mm" H 1195 5625 50  0001 C CNN
 F 3 "" H 1195 5625 50  0000 C CNN
 	1    1195 5625
@@
 F 0 "C2" H 1650 5885 50  0000 L CNN
 F 1 "100nF" H 1650 5685 50  0000 L CNN
-F 2 "Capacitors_THT:C_Disc_D5.0mm_W2.5mm_P5.00mm" H 1663 5635 50  0001 C CNN
+F 2 "Capacitors_SMD:C_1206_HandSoldering" H 1663 5635 50  0001 C CNN
 F 3 "" H 1625 5785 50  0000 C CNN
 	1    1625 5785
@@
 F 0 "R3" V 2165 5775 50  0000 C CNN
 F 1 "10k" V 2085 5775 50  0000 C CNN
-F 2 "Resistors_ThroughHole:Resistor_Horizontal_RM10mm" V 2015 5775 50  0001 C CNN
+F 2 "libreria_huellas_proyecto:Resistor_Horizontal_RM10mm" V 2015 5775 50  0001 C CNN
 F 3 "" H 2085 5775 50  0000 C CNN
 	1    2085 5775
@@
 F 0 "P3" H 3115 5775 50  0000 C CNN
 F 1 "PINZA_2" V 3215 5625 50  0000 C CNN
-F 2 "Connect:bornier2" H 3115 5625 50  0001 C CNN
+F 2 "Connectors_Terminal_Blocks:TerminalBlock_bornier-2_P5.08mm" H 3115 5625 50  0001 C CNN
 F 3 "" H 3115 5625 50  0000 C CNN
 	1    3115 5625
@@
 F 0 "C6" H 3570 5885 50  0000 L CNN
 F 1 "100nF" H 3570 5685 50  0000 L CNN
-F 2 "Capacitors_THT:C_Disc_D5.0mm_W2.5mm_P5.00mm" H 3583 5635 50  0001 C CNN
+F 2 "Capacitors_SMD:C_1206_HandSoldering" H 3583 5635 50  0001 C CNN
 F 3 "" H 3545 5785 50  0000 C CNN
 	1    3545 5785
@@
 F 0 "R5" V 4085 5775 50  0000 C CNN
 F 1 "10k" V 4005 5775 50  0000 C CNN
-F 2 "Resistors_ThroughHole:Resistor_Horizontal_RM10mm" V 3935 5775 50  0001 C CNN
+F 2 "libreria_huellas_proyecto:Resistor_Horizontal_RM10mm" V 3935 5775 50  0001 C CNN
 F 3 "" H 4005 5775 50  0000 C CNN
 	1    4005 5775
@@
 F 0 "P4" H 5035 5775 50  0000 C CNN
 F 1 "PINZA_3" V 5135 5625 50  0000 C CNN
-F 2 "Connect:bornier2" H 5035 5625 50  0001 C CNN
+F 2 "Connectors_Terminal_Blocks:TerminalBlock_bornier-2_P5.08mm" H 5035 5625 50  0001 C CNN
 F 3 "" H 5035 5625 50  0000 C CNN
 	1    5035 5625
@@
 F 0 "C8" H 5490 5885 50  0000 L CNN
 F 1 "100nF" H 5490 5685 50  0000 L CNN
-F 2 "Capacitors_THT:C_Disc_D5.0mm_W2.5mm_P5.00mm" H 5503 5635 50  0001 C CNN
+F 2 "Capacitors_SMD:C_1206_HandSoldering" H 5503 5635 50  0001 C CNN
 F 3 "" H 5465 5785 50  0000 C CNN
 	1    5465 5785
@@
 F 0 "R7" V 6005 5775 50  0000 C CNN
 F 1 "10k" V 5925 5775 50  0000 C CNN
-F 2 "Resistors_ThroughHole:Resistor_Horizontal_RM10mm" V 5855 5775 50  0001 C CNN
+F 2 "libreria_huellas_proyecto:Resistor_Horizontal_RM10mm" V 5855 5775 50  0001 C CNN
 F 3 "" H 5925 5775 50  0000 C CNN
 	1    5925 5775
@@
 F 0 "P5" H 6955 5775 50  0000 C CNN
 F 1 "PINZA_4" V 7055 5625 50  0000 C CNN
-F 2 "Connect:bornier2" H 6955 5625 50  0001 C CNN
+F 2 "Connectors_Terminal_Blocks:TerminalBlock_bornier-2_P5.08mm" H 6955 5625 50  0001 C CNN
 F 3 "" H 6955 5625 50  0000 C CNN
 	1    6955 5625
@@
 F 0 "C9" H 7410 5885 50  0000 L CNN
 F 1 "100nF" H 7410 5685 50  0000 L CNN
-F 2 "Capacitors_THT:C_Disc_D5.0mm_W2.5mm_P5.00mm" H 7423 5635 50  0001 C CNN
+F 2 "Capacitors_SMD:C_1206_HandSoldering" H 7423 5635 50  0001 C CNN
 F 3 "" H 7385 5785 50  0000 C CNN
 	1    7385 5785
@@
 F 0 "R8" V 7925 5775 50  0000 C CNN
 F 1 "10k" V 7845 5775 50  0000 C CNN
-F 2 "Resistors_ThroughHole:Resistor_Horizontal_RM10mm" V 7775 5775 50  0001 C CNN
+F 2 "libreria_huellas_proyecto:Resistor_Horizontal_RM10mm" V 7775 5775 50  0001 C CNN
 F 3 "" H 7845 5775 50  0000 C CNN
 	1    7845 5775
@@
 F 0 "P6" H 8920 5775 50  0000 C CNN
 F 1 "PINZA_5" V 9020 5625 50  0000 C CNN
-F 2 "Connect:bornier2" H 8920 5625 50  0001 C CNN
+F 2 "Connectors_Terminal_Blocks:TerminalBlock_bornier-2_P5.08mm" H 8920 5625 50  0001 C CNN
 F 3 "" H 8920 5625 50  0000 C CNN
 	1    8920 5625
@@
 F 0 "C11" H 9375 5885 50  0000 L CNN
 F 1 "100nF" H 9375 5685 50  0000 L CNN
-F 2 "Capacitors_THT:C_Disc_D5.0mm_W2.5mm_P5.00mm" H 9388 5635 50  0001 C CNN
+F 2 "Capacitors_SMD:C_1206_HandSoldering" H 9388 5635 50  0001 C CNN
 F 3 "" H 9350 5785 50  0000 C CNN
 	1    9350 5785
@@
 F 0 "R9" V 9890 5775 50  0000 C CNN
 F 1 "10k" V 9810 5775 50  0000 C CNN
-F 2 "Resistors_ThroughHole:Resistor_Horizontal_RM10mm" V 9740 5775 50  0001 C CNN
+F 2 "libreria_huellas_proyecto:Resistor_Horizontal_RM10mm" V 9740 5775 50  0001 C CNN
 F 3 "" H 9810 5775 50  0000 C CNN
 	1    9810 5775
@@
 F 0 "P7" H 1195 6735 50  0000 C CNN
 F 1 "PINZA_6" V 1295 6585 50  0000 C CNN
-F 2 "Connect:bornier2" H 1195 6585 50  0001 C CNN
+F 2 "Connectors_Terminal_Blocks:TerminalBlock_bornier-2_P5.08mm" H 1195 6585 50  0001 C CNN
 F 3 "" H 1195 6585 50  0000 C CNN
 	1    1195 6585
@@
 F 0 "C3" H 1650 6845 50  0000 L CNN
 F 1 "100nF" H 1650 6645 50  0000 L CNN
-F 2 "Capacitors_THT:C_Disc_D5.0mm_W2.5mm_P5.00mm" H 1663 6595 50  0001 C CNN
+F 2 "Capacitors_SMD:C_1206_HandSoldering" H 1663 6595 50  0001 C CNN
 F 3 "" H 1625 6745 50  0000 C CNN
 	1    1625 6745
@@
 F 0 "R4" V 2165 6735 50  0000 C CNN
 F 1 "10k" V 2085 6735 50  0000 C CNN
-F 2 "Resistors_ThroughHole:Resistor_Horizontal_RM10mm" V 2015 6735 50  0001 C CNN
+F 2 "libreria_huellas_proyecto:Resistor_Horizontal_RM10mm" V 2015 6735 50  0001 C CNN
 F 3 "" H 2085 6735 50  0000 C CNN
 	1    2085 6735
@@
 F 0 "P8" H 3115 6735 50  0000 C CNN
 F 1 "PINZA_7" V 3215 6585 50  0000 C CNN
-F 2 "Connect:bornier2" H 3115 6585 50  0001 C CNN
+F 2 "Connectors_Terminal_Blocks:TerminalBlock_bornier-2_P5.08mm" H 3115 6585 50  0001 C CNN
 F 3 "" H 3115 6585 50  0000 C CNN
 	1    3115 6585
@@
 F 0 "C7" H 3570 6845 50  0000 L CNN
 F 1 "100nF" H 3570 6645 50  0000 L CNN
-F 2 "Capacitors_THT:C_Disc_D5.0mm_W2.5mm_P5.00mm" H 3583 6595 50  0001 C CNN
+F 2 "Capacitors_SMD:C_1206_HandSoldering" H 3583 6595 50  0001 C CNN
 F 3 "" H 3545 6745 50  0000 C CNN
 	1    3545 6745
@@
 F 0 "R6" V 4085 6735 50  0000 C CNN
 F 1 "10k" V 4005 6735 50  0000 C CNN
-F 2 "Resistors_ThroughHole:Resistor_Horizontal_RM10mm" V 3935 6735 50  0001 C CNN
+F 2 "libreria_huellas_proyecto:Resistor_Horizontal_RM10mm" V 3935 6735 50  0001 C CNN
 F 3 "" H 4005 6735 50  0000 C CNN
 	1    4005 6735
@@
 F 0 "J4" H 8300 1760 50  0000 C CNN
 F 1 "Conn_02x05_Odd_Even" H 8300 1160 50  0000 C CNN
-F 2 "" H 8250 1460 50  0001 C CNN
+F 2 "Pin_Headers:Pin_Header_Straight_2x05_Pitch2.54mm" H 8250 1460 50  0001 C CNN
 F 3 "" H 8250 1460 50  0001 C CNN
 	1    8250 1460
@@
 F 0 "U1" H 2355 4210 50  0000 L CNN
 F 1 "LM358" H 2355 3810 50  0000 L CNN
-F 2 "" H 2355 4010 50  0001 C CNN
+F 2 "Housings_SOIC:SO-8_5.3x6.2mm_Pitch1.27mm" H 2355 4010 50  0001 C CNN
 F 3 "" H 2355 4010 50  0001 C CNN
 	1    2355 4010
@@
 P 1555 3705
 F 0 "R1" V 1635 3705 50  0000 C CNN
-F 1 "R" V 1555 3705 50  0000 C CNN
-F 2 "" V 1485 3705 50  0001 C CNN
+F 1 "4K7" V 1555 3705 50  0000 C CNN
+F 2 "Resistors_SMD:R_2512_HandSoldering" V 1485 3705 50  0001 C CNN
 F 3 "" H 1555 3705 50  0001 C CNN
 	1    1555 3705
@@
 P 1555 4090
 F 0 "R2" V 1635 4090 50  0000 C CNN
-F 1 "R" V 1555 4090 50  0000 C CNN
-F 2 "" V 1485 4090 50  0001 C CNN
+F 1 "4K7" V 1555 4090 50  0000 C CNN
+F 2 "Resistors_SMD:R_2512_HandSoldering" V 1485 4090 50  0001 C CNN
 F 3 "" H 1555 4090 50  0001 C CNN
 	1    1555 4090
@@
 F 0 "C10" H 8880 2945 50  0000 L CNN
 F 1 "100nF" H 8880 2745 50  0000 L CNN
-F 2 "Capacitors_THT:C_Disc_D5.0mm_W2.5mm_P5.00mm" H 8893 2695 50  0001 C CNN
+F 2 "Capacitors_SMD:C_1206_HandSoldering" H 8893 2695 50  0001 C CNN
 F 3 "" H 8855 2845 50  0000 C CNN
 	1    8855 2845
@@
 F 0 "C5" H 2995 4350 50  0000 L CNN
 F 1 "10uF" H 2995 4150 50  0000 L CNN
-F 2 "Capacitors_THT:CP_Radial_D5.0mm_P2.00mm" H 2970 4250 50  0001 C CNN
+F 2 "Capacitors_SMD:C_2220_HandSoldering" H 2970 4250 50  0001 C CNN
 F 3 "" H 2970 4250 50  0000 C CNN
 	1    2970 4250
@@
 F 0 "C1" H 1220 4160 50  0000 L CNN
 F 1 "10uF" H 1220 3960 50  0000 L CNN
-F 2 "Capacitors_THT:CP_Radial_D5.0mm_P2.00mm" H 1195 4060 50  0001 C CNN
+F 2 "Capacitors_SMD:C_2220_HandSoldering" H 1195 4060 50  0001 C CNN
 F 3 "" H 1195 4060 50  0000 C CNN
 	1    1195 4060
@@
 F 0 "P1" H 1090 2545 50  0000 C CNN
 F 1 "V_IN" V 1190 2395 50  0000 C CNN
-F 2 "Connect:bornier2" H 1090 2395 50  0001 C CNN
+F 2 "Connectors_Terminal_Blocks:TerminalBlock_bornier-2_P5.08mm" H 1090 2395 50  0001 C CNN
 F 3 "" H 1090 2395 50  0000 C CNN
 	1    1090 2395
@@
 F 0 "C4" H 2140 2695 50  0000 L CNN
 F 1 "10uF" H 2140 2495 50  0000 L CNN
-F 2 "Capacitors_THT:CP_Radial_D5.0mm_P2.00mm" H 2115 2595 50  0001 C CNN
+F 2 "Capacitors_SMD:C_2220_HandSoldering" H 2115 2595 50  0001 C CNN
 F 3 "" H 2115 2595 50  0000 C CNN
 	1    2115 2595
@@
 F 0 "D1" H 1840 2445 50  0000 C CNN
 F 1 "schottky" H 1840 2245 50  0000 C CNN
-F 2 "Diodes_ThroughHole:Diode_DO-35_SOD27_Horizontal_RM10" H 1840 2345 50  0001 C CNN
+F 2 "Diodes_SMD:D_2114" H 1840 2345 50  0001 C CNN
 F 3 "" H 1840 2345 50  0000 C CNN
 	1    1840 2345
@@
 F 0 "U2" H 5540 2920 50  0000 C CNN
 F 1 "NANO" H 5190 2770 50  0000 C CNN
-F 2 "oscar_libreria_huellas:arduino_nano" H 4890 1120 50  0001 C CNN
+F 2 "libreria_huellas_proyecto:arduino_nano" H 4890 1120 50  0001 C CNN
 F 3 "DOCUMENTATION" H 5040 1070 50  0001 C CNN
 	1    5190 1920

Commit message: desarrollo hardware
Parts:
- added C12, C13: 100nF, Capacitors_SMD:C_1206_HandSoldering, symbol C
- added R11, R12, R13: 4K7, Resistors_SMD:R_2512_HandSoldering, symbol R
Connections:
- wire segments 98 -> 105
- no-connect marks 20 -> 19
Other:
- moved on the sheet: C10, J1, J2, J3, J4

Commit message: avance en pcb
Connections:
- no-connect marks 19 -> 18

Commit message: hardware, rehubicacion de componentes
Parts:
- added J5: Conn_02x05_Odd_Even, oscar_libreria_huellas:Pin_Header_Straight_2x05_Pitch2.54mm_onsar, symbol Conn_02x05_Odd_Even
- J4: footprint Pin_Headers:Pin_Header_Straight_2x05_Pitch2.54mm -> oscar_libreria_huellas:Pin_Header_Straight_2x05_Pitch2.54mm_onsar
Connections:
- wire segments 105 -> 115
- no-connect marks 18 -> 21
Changed lines of the file:
@@
 F 3 "" H 1195 5625 50  0000 C CNN
 	1    1195 5625
-	-1   0    0    -1
+	-1   0    0    1
 $EndComp
 Text Label 2195 5990 0    60   ~ 0
@@
 F 3 "" H 3115 5625 50  0000 C CNN
 	1    3115 5625
-	-1   0    0    -1
+	-1   0    0    1
 $EndComp
 Text Label 4085 5575 0    60   ~ 0
@@
 F 3 "" H 5035 5625 50  0000 C CNN
 	1    5035 5625
-	-1   0    0    -1
+	-1   0    0    1
 $EndComp
 Text Label 6005 5575 0    60   ~ 0
@@
 F 3 "" H 6955 5625 50  0000 C CNN
 	1    6955 5625
-	-1   0    0    -1
+	-1   0    0    1
 $EndComp
 Text Label 7925 5575 0    60   ~ 0
@@
 F 3 "" H 8920 5625 50  0000 C CNN
 	1    8920 5625
-	-1   0    0    -1
+	-1   0    0    1
 $EndComp
 Text Label 9890 5575 0    60   ~ 0
@@
 F 3 "" H 1195 6585 50  0000 C CNN
 	1    1195 6585
-	-1   0    0    -1
+	-1   0    0    1
 $EndComp
 Text Label 2195 6950 0    60   ~ 0
@@
 F 3 "" H 3115 6585 50  0000 C CNN
 	1    3115 6585
-	-1   0    0    -1
+	-1   0    0    1
 $EndComp
 Text Label 4085 6535 0    60   ~ 0
@@
 F 0 "J4" H 7940 2240 50  0000 C CNN
 F 1 "Conn_02x05_Odd_Even" H 7940 1640 50  0000 C CNN
-F 2 "Pin_Headers:Pin_Header_Straight_2x05_Pitch2.54mm" H 7890 1940 50  0001 C CNN
+F 2 "oscar_libreria_huellas:Pin_Header_Straight_2x05_Pitch2.54mm_onsar" H 7890 1940 50  0001 C CNN
 F 3 "" H 7890 1940 50  0001 C CNN
 	1    7890 1940
@@
 F 3 "" H 1090 2395 50  0000 C CNN
 	1    1090 2395
-	-1   0    0    -1
+	-1   0    0    1
 $EndComp
 $Comp
@@
 	7690 2140 7455 2140
 NoConn ~ 7255 1840
+$Comp
+L Conn_02x05_Odd_Even J5
+U 1 1 5D6D477F
+P 7905 2740
+F 0 "J5" H 7955 3040 50  0000 C CNN
+F 1 "Conn_02x05_Odd_Even" H 7955 2440 50  0000 C CNN
+F 2 "oscar_libreria_huellas:Pin_Header_Straight_2x05_Pitch2.54mm_onsar" H 7905 2740 50  0001 C CNN
+F 3 "" H 7905 2740 50  0001 C CNN
+	1    7905 2740
+	1    0    0    -1
+$EndComp
+Text Label 8240 2840 0    60   ~ 0
+mosi
+Text Label 8240 2940 0    60   ~ 0
+miso
+Text Label 7470 2940 0    60   ~ 0
+sck
+Text Label 8240 2740 0    60   ~ 0
+esp_d0
+Text Label 8235 2640 0    60   ~ 0
+esp_d1
+Text Label 8235 2540 0    60   ~ 0
+esp_d2
+$Comp
+L GND #PWR015
+U 1 1 5D6D478C
+P 7270 2840
+F 0 "#PWR015" H 7270 2590 50  0001 C CNN
+F 1 "GND" H 7270 2690 50  0000 C CNN
+F 2 "" H 7270 2840 50  0001 C CNN
+F 3 "" H 7270 2840 50  0001 C CNN
+	1    7270 2840
+	1    0    0    -1
+$EndComp
+NoConn ~ 7270 2740
+Wire Wire Line
+	8205 2740 8640 2740
+Wire Wire Line
+	8205 2940 8640 2940
+Wire Wire Line
+	7270 2540 7705 2540
+Wire Wire Line
+	7270 2640 7705 2640
+Wire Wire Line
+	7270 2740 7705 2740
+Wire Wire Line
+	7270 2840 7705 2840
+Wire Wire Line
+	8205 2540 8640 2540
+Wire Wire Line
+	8205 2640 8640 2640
+Wire Wire Line
+	8205 2840 8640 2840
+Wire Wire Line
+	7705 2940 7470 2940
+NoConn ~ 7270 2640
+NoConn ~ 7270 2540
 $EndSCHEMATC

Commit message: desarrollo hardware
Parts:
- removed C7: 100nF, Capacitors_SMD:C_1206_HandSoldering, symbol C
- added R10: 10k, Resistors_SMD:R_1206_HandSoldering, symbol R
- R1, R11, R12, R13, R2: footprint Resistors_SMD:R_2512_HandSoldering -> Resistors_SMD:R_1206_HandSoldering
- R6: value 10k -> 1k
Connections:
- net labels added: voltage_1
- net labels removed: intensidad_7
- wire segments 115 -> 114
Changed lines of the file:
@@
 encoding utf-8
 Sheet 1 1
-Title ""
+Title "EcoPower"
 Date ""
 Rev ""
-Comp ""
+Comp "iotlibre"
 Comment1 ""
 Comment2 ""
@@
 	-1   0    0    1
 $EndComp
-Text Label 4085 6535 0    60   ~ 0
-intensidad_7
 Text Label 4115 6950 0    60   ~ 0
 v_referencia
-$Comp
-L C C7
-U 1 1 5D4C6F33
-P 3545 6745
-F 0 "C7" H 3570 6845 50  0000 L CNN
-F 1 "100nF" H 3570 6645 50  0000 L CNN
-F 2 "Capacitors_SMD:C_1206_HandSoldering" H 3583 6595 50  0001 C CNN
-F 3 "" H 3545 6745 50  0000 C CNN
-	1    3545 6745
-	1    0    0    -1
-$EndComp
 $Comp
 L R R6
@@
 P 4005 6735
 F 0 "R6" V 4085 6735 50  0000 C CNN
-F 1 "10k" V 4005 6735 50  0000 C CNN
+F 1 "1k" V 4005 6735 50  0000 C CNN
 F 2 "libreria_huellas_proyecto:Resistor_Horizontal_RM10mm" V 3935 6735 50  0001 C CNN
 F 3 "" H 4005 6735 50  0000 C CNN
@@
 F 0 "R1" V 1635 3705 50  0000 C CNN
 F 1 "4K7" V 1555 3705 50  0000 C CNN
-F 2 "Resistors_SMD:R_2512_HandSoldering" V 1485 3705 50  0001 C CNN
+F 2 "Resistors_SMD:R_1206_HandSoldering" V 1485 3705 50  0001 C CNN
 F 3 "" H 1555 3705 50  0001 C CNN
 	1    1555 3705
@@
 F 0 "R2" V 1635 4090 50  0000 C CNN
 F 1 "4K7" V 1555 4090 50  0000 C CNN
-F 2 "Resistors_SMD:R_2512_HandSoldering" V 1485 4090 50  0001 C CNN
+F 2 "Resistors_SMD:R_1206_HandSoldering" V 1485 4090 50  0001 C CNN
 F 3 "" H 1555 4090 50  0001 C CNN
 	1    1555 4090
@@
 Text Label 6010 1820 0    60   ~ 0
 intensidad_6
-Text Label 6010 1720 0    60   ~ 0
-intensidad_7
 Text Label 6000 1620 0    60   ~ 0
 v_referencia
@@
 F 0 "R12" V 9570 1855 50  0000 C CNN
 F 1 "4K7" V 9490 1855 50  0000 C CNN
-F 2 "Resistors_SMD:R_2512_HandSoldering" V 9420 1855 50  0001 C CNN
+F 2 "Resistors_SMD:R_1206_HandSoldering" V 9420 1855 50  0001 C CNN
 F 3 "" H 9490 1855 50  0001 C CNN
 	1    9490 1855
@@
 F 0 "R11" V 9215 1065 50  0000 C CNN
 F 1 "4K7" V 9135 1065 50  0000 C CNN
-F 2 "Resistors_SMD:R_2512_HandSoldering" V 9065 1065 50  0001 C CNN
+F 2 "Resistors_SMD:R_1206_HandSoldering" V 9065 1065 50  0001 C CNN
 F 3 "" H 9135 1065 50  0001 C CNN
 	1    9135 1065
@@
 F 0 "R13" V 9975 2605 50  0000 C CNN
 F 1 "4K7" V 9895 2605 50  0000 C CNN
-F 2 "Resistors_SMD:R_2512_HandSoldering" V 9825 2605 50  0001 C CNN
+F 2 "Resistors_SMD:R_1206_HandSoldering" V 9825 2605 50  0001 C CNN
 F 3 "" H 9895 2605 50  0001 C CNN
 	1    9895 2605
@@
 Wire Wire Line
 	3315 6635 3315 6950
-Wire Wire Line
-	3315 6535 4365 6535
 Connection ~ 4005 6535
 Wire Wire Line
 	4005 6585 4005 6535
-Connection ~ 3545 6535
-Wire Wire Line
-	3545 6595 3545 6535
 Wire Wire Line
 	8190 1940 8625 1940
@@
 	2085 6885 2085 6950
 Connection ~ 2085 6950
-Wire Wire Line
-	3545 6895 3545 6950
-Connection ~ 3545 6950
 Wire Wire Line
 	4005 6885 4005 6950
@@
 NoConn ~ 7270 2640
 NoConn ~ 7270 2540
+Text Label 4120 6535 0    60   ~ 0
+voltage_1
+$Comp
+L R R10
+U 1 1 5D7208D8
+P 3625 6535
+F 0 "R10" V 3705 6535 50  0000 C CNN
+F 1 "10k" V 3625 6535 50  0000 C CNN
+F 2 "Resistors_SMD:R_1206_HandSoldering" V 3555 6535 50  0001 C CNN
+F 3 "" H 3625 6535 50  0000 C CNN
+	1    3625 6535
+	0    1    1    0
+$EndComp
+Wire Wire Line
+	3315 6535 3475 6535
+Wire Wire Line
+	3775 6535 4365 6535
+Text Label 6000 1720 0    60   ~ 0
+voltage_1
 $EndSCHEMATC

Commit message: primera version hardware esclavo
Parts:
- added unit 2 of U1
Connections:
- net labels added: v_25
- wire segments 114 -> 121
Changed lines of the file:
@@
 Text Label 6000 1720 0    60   ~ 0
 voltage_1
+$Comp
+L LM358 U1
+U 2 1 5D755B03
+P 5115 4065
+F 0 "U1" H 5115 4265 50  0000 L CNN
+F 1 "LM358" H 5115 3865 50  0000 L CNN
+F 2 "Housings_SOIC:SO-8_5.3x6.2mm_Pitch1.27mm" H 5115 4065 50  0001 C CNN
+F 3 "" H 5115 4065 50  0001 C CNN
+	2    5115 4065
+	1    0    0    -1
+$EndComp
+Wire Wire Line
+	5015 3765 5015 3655
+Text Label 5015 3655 0    60   ~ 0
+vin_5V
+$Comp
+L GND #PWR016
+U 1 1 5D7561B7
+P 5015 4365
+F 0 "#PWR016" H 5015 4115 50  0001 C CNN
+F 1 "GND" H 5015 4215 50  0000 C CNN
+F 2 "" H 5015 4365 50  0000 C CNN
+F 3 "" H 5015 4365 50  0000 C CNN
+	1    5015 4365
+	-1   0    0    -1
+$EndComp
+Wire Wire Line
+	4815 4165 4660 4165
+Wire Wire Line
+	4660 4165 4660 4580
+Wire Wire Line
+	4660 4580 5480 4580
+Wire Wire Line
+	5480 4580 5480 4065
+Wire Wire Line
+	5480 4065 5415 4065
+Text Label 1635 3910 0    60   ~ 0
+v_25
+Wire Wire Line
+	4815 3965 4455 3965
+Text Label 4455 3965 0    60   ~ 0
+v_25
 $EndSCHEMATC
