File: hardware/iot_esp/iotesp_modbus_hardware/ecoBeat_3.sch (KiCad schematic (older format))
At the start: 6 parts, among them P1 CONN_02X05, U1 WeMos_mini

Commit message: avances en hardware de master
Parts:
- added D3: Schottky, Diodes_THT:D_DO-35_SOD27_P10.16mm_Horizontal, symbol D_Schottky
- added J1: Test, Wire_Pads:SolderWirePad_single_0-8mmDrill, symbol TEST_1P
- D1: footprint LEDs:LED_1206 -> LEDs:LED_D3.0mm
- D2: renamed from D3; footprint LEDs:LED_1206 -> LEDs:LED_D3.0mm
- R1: renamed from R6; footprint Resistors_SMD:R_1206 -> Resistors_THT:R_Axial_DIN0207_L6.3mm_D2.5mm_P10.16mm_Horizontal
- R2: renamed from R8; footprint Resistors_SMD:R_1206 -> Resistors_THT:R_Axial_DIN0207_L6.3mm_D2.5mm_P10.16mm_Horizontal
Connections:
- net labels added: vin_5v
- wire segments 30 -> 33
Other:
- moved on the sheet: D1, D2, P1, R1, R2, U1
