File: hardware/iot_esp/iotesp_modbus_hardware/ecoBeat_3.kicad_pcb (KiCad board)
At the start: 2 copper layers, 6 parts, among them P1 CONN_02X05, U1 WeMos_mini

Commit message: avances en hardware de master
Parts:
- removed R6, R8: 220, Resistors_SMD:R_1206
- added D2: LED, LEDs:LED_D3.0mm, F.Cu at (102.6, 53.1)
- added J1: Test, Wire_Pads:SolderWirePad_single_0-8mmDrill, F.Cu at (97.0, 52.5)
- added R1: 220, Resistors_THT:R_Axial_DIN0207_L6.3mm_D2.5mm_P10.16mm_Horizontal, F.Cu at (104.6, 65.7)
- added R2: 220, Resistors_THT:R_Axial_DIN0207_L6.3mm_D2.5mm_P10.16mm_Horizontal, F.Cu at (104.6, 60.6)
- D1: footprint LEDs:LED_1206 -> LEDs:LED_D3.0mm
- D3: value LED -> Schottky; footprint LEDs:LED_1206 -> Diodes_THT:D_DO-35_SOD27_P10.16mm_Horizontal
- P1: moved to B.Cu
- moved P1 147.2 mm to (50.4, 61.0), turned to 270 degrees
- moved U1 98.0 mm to (78.4, 70.7)
- moved D3 74.5 mm to (86.2, 62.6), turned to 180 degrees
- moved D1 63.9 mm to (108.6, 53.1), turned to 180 degrees
Connections:
- D3 pad 1: GND -> /vin_5v
- D3 pad 2: Net-(D3-Pad2) -> /vcc_5v
- U1 pad 9: /vcc_5v -> /vin_5v
Routing:
- net /esp_d2: track 0.00 -> 78.2 mm
- net /esp_d1: track 0.00 -> 59.9 mm
- net /mosi: track 0.00 -> 54.2 mm
- net /miso: track 0.00 -> 41.7 mm
- net /esp_d3: track 0.00 -> 40.4 mm
- net /vcc_5v: track 0.00 -> 31.0 mm
- net /esp_d0: track 0.00 -> 18.8 mm, vias 0 -> 1
- net /esp_d8: track 0.00 -> 18.7 mm
- net /sck: track 0.00 -> 14.6 mm
- net Net-(D1-Pad2): track 0.00 -> 13.8 mm
- net Net-(D2-Pad2): track 0.00 -> 10.7 mm
- net /esp_d4: track 0.00 -> 4.64 mm
- net /vin_5v: track 0.00 -> 4.57 mm

Commit message: desarrollo pcb master
Parts:
- moved J1 1.48 mm to (95.6, 52.9)
Routing:
- net GND: track 0.00 -> 100.8 mm
- net /esp_d2: track 78.2 -> 54.1 mm
- net /vin_5v: track 4.57 -> 17.1 mm
- net /vcc_5v: track 31.0 -> 34.3 mm
- net /esp_d8: track 18.7 -> 21.7 mm, vias 0 -> 1
- net /esp_d1: track 59.9 -> 59.2 mm
