File: hardware/iot_esp/iotesp_hardware/ecoBeat_3.sch (KiCad schematic (older format))
At the start: 8 parts, among them J1 Test, P1 CONN_02X05, U1 WeMos_mini

Commit message: PCB iot_esp12 v2 enviada a fabricar
Parts:
- added R1, R2, R3, R4: 10K, Resistors_SMD:R_1206_HandSoldering, symbol R
- added R5, R6: 20K, Resistors_SMD:R_1206_HandSoldering, symbol R
- added R7: 120, Resistors_SMD:R_1206_HandSoldering, symbol R
- added U2: MAX_485, SMD_Packages:SOIC-8-N, symbol MAX_485
- D1: renamed from D3; footprint Diodes_THT:D_DO-35_SOD27_P10.16mm_Horizontal -> Diodes_SMD:D_2114; symbol D_Schottky -> D_Schottky-RESCUE-ecoBeat_3
- P1: footprint oscar_libreria:Pin_Header_Straight_2x05_Pitch2.54mm_onsar -> libreria_huellas_proyecto:D1_mini_board
- R8: renamed from R1; footprint Resistors_THT:R_Axial_DIN0207_L6.3mm_D2.5mm_P10.16mm_Horizontal -> Resistors_SMD:R_1206_HandSoldering
- R9: renamed from R2; footprint Resistors_THT:R_Axial_DIN0207_L6.3mm_D2.5mm_P10.16mm_Horizontal -> Resistors_SMD:R_1206_HandSoldering
- U1: footprint wemos_d1_mini:D1_mini_board -> libreria_huellas_proyecto:D1_mini_board_oscar
- renumbered D1 to D2, D2 to D3
Connections:
- net labels added: esp_d5, esp_d6, esp_rx, esp_rx2, esp_tx, esp_tx2, mb_a, mb_b
- net labels removed: esp_d1, esp_d3, esp_d8, miso, mosi, sck
- wire segments 33 -> 57
Other:
- moved on the sheet: D1, D2, D3, J1, P1, R8, R9, U1
